File: nix-pill-v1.sch (KiCad schematic (older format))
At the start: 40 parts, among them J1 LEFT, J2 BOOT, J3 RIGHT, J4 SWD, J5 USB_B_Micro, SW1 USER0, SW2 NRST, U1 AMS1117-3.3, U2 STM32F103C8Tx, Y1 32.768KHz LSE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

Commit message: Started adding data sheets Started the BOM Calculated the LED limiting R
Parts:
- R1, R2: value 510 -> 100
Changed lines of the file:
@@
 P 1800 1550
 F 0 "R2" V 2000 1500 50  0000 L CNN
-F 1 "510" V 1900 1500 50  0000 L CNN
+F 1 "100" V 1900 1500 50  0000 L CNN
 F 2 "Resistor_SMD:R_0603_1608Metric" H 1800 1550 50  0001 C CNN
 F 3 "~" H 1800 1550 50  0001 C CNN
@@
 P 1800 1200
 F 0 "R1" V 2000 1150 50  0000 L CNN
-F 1 "510" V 1900 1150 50  0000 L CNN
+F 1 "100" V 1900 1150 50  0000 L CNN
 F 2 "Resistor_SMD:R_0603_1608Metric" H 1800 1200 50  0001 C CNN
 F 3 "~" H 1800 1200 50  0001 C CNN

Commit message: Added more data sheets and updated BOM
Parts:
- C3, C6: value 20pF -> 10pF
Changed lines of the file:
@@
 P 4900 2300
 F 0 "C3" H 4700 2350 50  0000 L CNN
-F 1 "20pF" H 4650 2250 50  0000 L CNN
+F 1 "10pF" H 4650 2250 50  0000 L CNN
 F 2 "Capacitor_SMD:C_0603_1608Metric" H 4900 2300 50  0001 C CNN
 F 3 "~" H 4900 2300 50  0001 C CNN
@@
 P 5400 2300
 F 0 "C6" H 5492 2346 50  0000 L CNN
-F 1 "20pF" H 5492 2255 50  0000 L CNN
+F 1 "10pF" H 5492 2255 50  0000 L CNN
 F 2 "Capacitor_SMD:C_0603_1608Metric" H 5400 2300 50  0001 C CNN
 F 3 "~" H 5400 2300 50  0001 C CNN

Commit message: BOM completed. Ordering PCB and parts
Parts:
- C2, C5: value 20pF -> 8pF
- R9: value 10M -> 1M
Changed lines of the file:
@@
 P 5400 2050
 F 0 "R9" H 5459 2096 50  0000 L CNN
-F 1 "10M" H 5459 2005 50  0000 L CNN
+F 1 "1M" H 5459 2005 50  0000 L CNN
 F 2 "Resistor_SMD:R_0603_1608Metric" H 5400 2050 50  0001 C CNN
 F 3 "~" H 5400 2050 50  0001 C CNN
@@
 P 5400 1500
 F 0 "C5" H 5492 1546 50  0000 L CNN
-F 1 "20pF" H 5492 1455 50  0000 L CNN
+F 1 "8pF" H 5492 1455 50  0000 L CNN
 F 2 "Capacitor_SMD:C_0603_1608Metric" H 5400 1500 50  0001 C CNN
 F 3 "~" H 5400 1500 50  0001 C CNN
@@
 P 4900 1500
 F 0 "C2" H 4700 1550 50  0000 L CNN
-F 1 "20pF" H 4650 1450 50  0000 L CNN
+F 1 "8pF" H 4650 1450 50  0000 L CNN
 F 2 "Capacitor_SMD:C_0603_1608Metric" H 4900 1500 50  0001 C CNN
 F 3 "~" H 4900 1500 50  0001 C CNN
