File: nix-pill-v1.kicad_pcb (KiCad board)
At the start: 2 copper layers, 75 x 35 mm, 40 parts, among them J1 LEFT, J2 BOOT, J3 RIGHT, J4 SWD, J5 USB_B_Micro, SW1 USER0, SW2 NRST, U1 AMS1117-3.3, U2 STM32F103C8Tx, Y1 32.768KHz LSE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

Commit message: Set the board clearance to match board house.
Other:
- net class Default: clearance 0.2 -> 0.127
- rule trace_clearance: 0.2 -> 0.127
- rule trace_min: 0.2 -> 0.02
